File: uOsc_2 board_2_v2.0.sch (EAGLE design)
At the start: 154 parts, among them IC1 R-78E3.3-0.5, IC2 TLC59281DBQ, IC3 LD2981ABU33, IC4 STM32F373CCT6, IC5 PCM5100APW, IC6 MCP6004, IC7 MCP6004, IC8 TL072PW, IC9 LM4040B10, Q1 8MHz

Commit message: uOsc-II files
Other:
- note added: "Codex-Modulex"
- note added: "Original design by: Olivier Gillet of Mutable Instruments"
- note added: "info@codex-modulex.com"
- note removed: "Olivier Gillet"
- note removed: "ol.gillet@gmail.com"
- moved on the sheet: FREQ_ATT, MORPH_ATT, MORPH_POT, SW1, SW2, TIMBRE_ATT, TIMBRE_POT
